Commit message: new-dobot-api-timeout

File: services/robot_container/ros_ws/src/OrbbecSDK_ROS2/orbbec_description/urdf/gemini_335_336.urdf.xacro (robot description, xacro)
@@ -15,5 +15,5 @@
         </inertial>
         <visual>
-            <origin xyz="0 0 0" rpy="0 0 0" />
+            <origin xyz="-0.01587 -0.025 -0.0125" rpy="0 0 0" />
             <geometry>
                 <mesh filename="${mesh_path}camera_link.STL" />
@@ -55,10 +55,10 @@
     </link>
     <joint name="camera_bottom_screw_frame_joint" type="fixed">
-        <origin xyz="0 0 0" rpy="0 0 0" />
+        <origin xyz="-0.01587 -0.025 -0.0125" rpy="0 0 0" />
         <parent link="camera_link" />
         <child link="camera_bottom_screw_frame" />
         <axis xyz="0 0 0" />
     </joint>
-    <link name="camera_infra_1_frame">
+    <link name="camera_left_ir_frame">
         <inertial>
             <origin xyz="-0.00158020887627678 -1.52683853303637E-08 -1.4860800305164E-07"
@@ -70,26 +70,26 @@
         </inertial>
         <visual>
-            <origin xyz="0 0 0" rpy="0 0 0" />
-            <geometry>
-                <mesh filename="${mesh_path}camera_infra_1_frame.STL" />
-            </geometry>
-            <material name="">
-                <color rgba="0.501960784313725 0.250980392156863 0.250980392156863 1" />
-            </material>
-        </visual>
-        <collision>
-            <origin xyz="0 0 0" rpy="0 0 0" />
-            <geometry>
-                <mesh filename="${mesh_path}camera_infra_1_frame.STL" />
-            </geometry>
-        </collision>
-    </link>
-    <joint name="camera_infra_1_joint" type="fixed">
-        <origin xyz="0.01587 -0.025 0.0125" rpy="0 0 0" />
-        <parent link="camera_bottom_screw_frame" />
-        <child link="camera_infra_1_frame" />
-        <axis xyz="0 0 0" />
-    </joint>
-    <link name="camera_infra_1_optical_frame">
+            <origin xyz="-25 0 0" rpy="0 0 0" />
+            <geometry>
+                <mesh filename="${mesh_path}camera_left_ir_frame.STL" />
+            </geometry>
+            <material name="">
+                <color rgba="0.501960784313725 0.250980392156863 0.250980392156863 1" />
+            </material>
+        </visual>
+        <collision>
+            <origin xyz="0 0 0" rpy="0 0 0" />
+            <geometry>
+                <mesh filename="${mesh_path}camera_left_ir_frame.STL" />
+            </geometry>
+        </collision>
+    </link>
+    <joint name="camera_left_ir_joint" type="fixed">
+        <origin xyz="0 0 0" rpy="0 0 0" />
+        <parent link="camera_depth_frame" />
+        <child link="camera_left_ir_frame" />
+        <axis xyz="0 0 0" />
+    </joint>
+    <link name="camera_left_ir_optical_frame">
         <inertial>
             <origin xyz="1.52683853338331E-08 1.48608003051636E-07 -0.00158020887627678" rpy="0 0 0" />
@@ -102,24 +102,24 @@
             <origin xyz="0 0 0" rpy="0 0 0" />
             <geometry>
-                <mesh filename="${mesh_path}camera_infra_1_optical_frame.STL" />
-            </geometry>
-            <material name="">
-                <color rgba="0.501960784313725 0.250980392156863 0.250980392156863 1" />
-            </material>
-        </visual>
-        <collision>
-            <origin xyz="0 0 0" rpy="0 0 0" />
-            <geometry>
-                <mesh filename="${mesh_path}camera_infra_1_optical_frame.STL" />
-            </geometry>
-        </collision>
-    </link>
-    <joint name="camera_infra_1_optical_joint" type="fixed">
-        <origin xyz="0.01587 -0.025 0.0125" rpy="-1.5707963267949 0 -1.5707963267949" />
-        <parent link="camera_bottom_screw_frame" />
-        <child link="camera_infra_1_optical_frame" />
-        <axis xyz="0 0 0" />
-    </joint>
-    <link name="camera_infra2_frame">
+                <mesh filename="${mesh_path}camera_left_ir_optical_frame.STL" />
+            </geometry>
+            <material name="">
+                <color rgba="0.501960784313725 0.250980392156863 0.250980392156863 1" />
+            </material>
+        </visual>
+        <collision>
+            <origin xyz="0 0 0" rpy="0 0 0" />
+            <geometry>
+                <mesh filename="${mesh_path}camera_left_ir_optical_frame.STL" />
+            </geometry>
+        </collision>
+    </link>
+    <joint name="camera_left_ir_optical_joint" type="fixed">
+        <origin xyz="0 0 0" rpy="-1.5707963267949 0 -1.5707963267949" />
+        <parent link="camera_left_ir_frame" />
+        <child link="camera_left_ir_optical_frame" />
+        <axis xyz="0 0 0" />
+    </joint>
+    <link name="camera_right_ir_frame">
         <inertial>
             <origin xyz="-0.00158020887627678 -1.52683853303637E-08 -1.48608003050581E-07"
@@ -133,24 +133,24 @@
             <origin xyz="0 0 0" rpy="0 0 0" />
             <geometry>
-                <mesh filename="${mesh_path}camera_infra2_frame.STL" />
-            </geometry>
-            <material name="">
-                <color rgba="0.501960784313725 0.250980392156863 0.250980392156863 1" />
-            </material>
-        </visual>
-        <collision>
-            <origin xyz="0 0 0" rpy="0 0 0" />
-            <geometry>
-                <mesh filename="${mesh_path}camera_infra2_frame.STL" />
-            </geometry>
-        </collision>
-    </link>
-    <joint name="camera_infra2_joint" type="fixed">
-        <origin xyz="0.01587 0.025 0.0125" rpy="0 0 0" />
-        <parent link="camera_bottom_screw_frame" />
-        <child link="camera_infra2_frame" />
-        <axis xyz="0 0 0" />
-    </joint>
-    <link name="camera_infra2_optical_frame">
+                <mesh filename="${mesh_path}camera_right_ir_frame.STL" />
+            </geometry>
+            <material name="">
+                <color rgba="0.501960784313725 0.250980392156863 0.250980392156863 1" />
+            </material>
+        </visual>
+        <collision>
+            <origin xyz="0 0 0" rpy="0 0 0" />
+            <geometry>
+                <mesh filename="${mesh_path}camera_right_ir_frame.STL" />
+            </geometry>
+        </collision>
+    </link>
+    <joint name="camera_right_ir_joint" type="fixed">
+        <origin xyz="0 -0.05 0" rpy="0 0 0" />
+        <parent link="camera_depth_frame" />
+        <child link="camera_right_ir_frame" />
+        <axis xyz="0 0 0" />
+    </joint>
+    <link name="camera_right_ir_optical_frame">
         <inertial>
             <origin xyz="1.52683853268942E-08 1.4860800305058E-07 -0.00158020887627678" rpy="0 0 0" />
@@ -163,21 +163,21 @@
             <origin xyz="0 0 0" rpy="0 0 0" />
             <geometry>
-                <mesh filename="${mesh_path}camera_infra2_optical_frame.STL" />
-            </geometry>
-            <material name="">
-                <color rgba="0.501960784313725 0.250980392156863 0.250980392156863 1" />
-            </material>
-        </visual>
-        <collision>
-            <origin xyz="0 0 0" rpy="0 0 0" />
-            <geometry>
-                <mesh filename="${mesh_path}camera_infra2_optical_frame.STL" />
-            </geometry>
-        </collision>
-    </link>
-    <joint name="camera_infra2_optical_joint" type="fixed">
-        <origin xyz="0.01587 0.025 0.0125" rpy="-1.5707963267949 0 -1.5707963267949" />
-        <parent link="camera_bottom_screw_frame" />
-        <child link="camera_infra2_optical_frame" />
+                <mesh filename="${mesh_path}camera_right_ir_optical_frame.STL" />
+            </geometry>
+            <material name="">
+                <color rgba="0.501960784313725 0.250980392156863 0.250980392156863 1" />
+            </material>
+        </visual>
+        <collision>
+            <origin xyz="0 0 0" rpy="0 0 0" />
+            <geometry>
+                <mesh filename="${mesh_path}camera_right_ir_optical_frame.STL" />
+            </geometry>
+        </collision>
+    </link>
+    <joint name="camera_right_ir_optical_joint" type="fixed">
+        <origin xyz="0 0 0" rpy="-1.5707963267949 0 -1.5707963267949" />
+        <parent link="camera_right_ir_frame" />
+        <child link="camera_right_ir_optical_frame" />
         <axis xyz="0 0 0" />
     </joint>
@@ -208,6 +208,6 @@
     </link>
     <joint name="camera_color_joint" type="fixed">
-        <origin xyz="0.017533 0.010995 0.012505" rpy="0 0 0" />
-        <parent link="camera_bottom_screw_frame" />
+        <origin xyz="0.001663 -0.014005 0.000005" rpy="0 0 0" />
+        <parent link="camera_depth_frame" />
         <child link="camera_color_frame" />
         <axis xyz="0 0 0" />
@@ -239,6 +239,6 @@
     </link>
     <joint name="camera_color_optical_joint" type="fixed">
-        <origin xyz="0.017533 0.010995 0.012505" rpy="-1.5707963267949 0 -1.5707963267949" />
-        <parent link="camera_bottom_screw_frame" />
+        <origin xyz="0 0 0" rpy="-1.5707963267949 0 -1.5707963267949" />
+        <parent link="camera_color_frame" />
         <child link="camera_color_optical_frame" />
         <axis xyz="0 0 0" />
@@ -270,6 +270,6 @@
     </link>
     <joint name="camera_depth_joint" type="fixed">
-        <origin xyz="0.01587 -0.025 0.0125" rpy="0 0 0" />
-        <parent link="camera_bottom_screw_frame" />
+        <origin xyz="0 0 0" rpy="0 0 0" />
+        <parent link="camera_link" />
         <child link="camera_depth_frame" />
         <axis xyz="0 0 0" />
@@ -299,6 +299,6 @@
     </link>
     <joint name="camera_depth_optical_joint" type="fixed">
-        <origin xyz="0.01587 -0.025 0.0125" rpy="-1.5707963267949 0 -1.5707963267949" />
-        <parent link="camera_bottom_screw_frame" />
+        <origin xyz="0 0 0" rpy="-1.5707963267949 0 -1.5707963267949" />
+        <parent link="camera_depth_frame" />
         <child link="camera_depth_optical_frame" />
         <axis xyz="0 0 0" />

File: services/robot_container/ros_ws/src/OrbbecSDK_ROS2/orbbec_description/urdf/test_astra2.urdf.xacro (robot description, xacro)
@@ -3,6 +3,6 @@
      Commit Version: 1.6.0-4-g7f85cfe  Build Version: 1.6.7995.38578
      For more information, please see http://wiki.ros.org/sw_urdf_exporter -->
-<robot name="gemini_336" xmlns:xacro="http://ros.org/wiki/xacro">
-    <xacro:include filename="gemini_335_336.urdf.xacro"/>
+<robot name="astra2" xmlns:xacro="http://ros.org/wiki/xacro">
+    <xacro:include filename="astra2.urdf.xacro"/>
     <!-- Define a virtual root link -->
   <link name="base_link"/>
@@ -11,5 +11,5 @@
     <parent link="base_link"/>
     <child link="camera_link"/>
-    <origin xyz="0.01587 0.025 0.0125" rpy="0 0 0"/>
+    <origin xyz="0.012323996052145958 0.03750000149011612 0.028150320053100586" rpy="0 0 0"/>
   </joint>
 </robot>

File: services/robot_container/ros_ws/src/OrbbecSDK_ROS2/orbbec_description/urdf/test_gemini2.urdf.xacro (robot description, xacro)
@@ -3,6 +3,6 @@
      Commit Version: 1.6.0-4-g7f85cfe  Build Version: 1.6.7995.38578
      For more information, please see http://wiki.ros.org/sw_urdf_exporter -->
-<robot name="gemini_336" xmlns:xacro="http://ros.org/wiki/xacro">
-    <xacro:include filename="gemini_335_336.urdf.xacro"/>
+<robot name="gemini2" xmlns:xacro="http://ros.org/wiki/xacro">
+    <xacro:include filename="gemini2.urdf.xacro"/>
     <!-- Define a virtual root link -->
   <link name="base_link"/>
@@ -11,5 +11,5 @@
     <parent link="base_link"/>
     <child link="camera_link"/>
-    <origin xyz="0.01587 0.025 0.0125" rpy="0 0 0"/>
+    <origin xyz="0.01491 0.025 0.0125" rpy="0 0 0"/>
   </joint>
 </robot>

File: services/robot_container/ros_ws/src/OrbbecSDK_ROS2/orbbec_description/urdf/test_gemini2L.urdf.xacro (robot description, xacro)
@@ -3,6 +3,6 @@
      Commit Version: 1.6.0-4-g7f85cfe  Build Version: 1.6.7995.38578
      For more information, please see http://wiki.ros.org/sw_urdf_exporter -->
-<robot name="gemini_336" xmlns:xacro="http://ros.org/wiki/xacro">
-    <xacro:include filename="gemini_335_336.urdf.xacro"/>
+<robot name="gemini2L" xmlns:xacro="http://ros.org/wiki/xacro">
+    <xacro:include filename="gemini2L.urdf.xacro"/>
     <!-- Define a virtual root link -->
   <link name="base_link"/>
@@ -11,5 +11,5 @@
     <parent link="base_link"/>
     <child link="camera_link"/>
-    <origin xyz="0.01587 0.025 0.0125" rpy="0 0 0"/>
+    <origin xyz="0.01033 0.05 0.0145" rpy="0 0 0"/>
   </joint>
 </robot>

File: services/robot_container/ros_ws/src/OrbbecSDK_ROS2/orbbec_description/urdf/test_gemini335L.urdf.xacro (robot description, xacro)
@@ -3,6 +3,6 @@
      Commit Version: 1.6.0-4-g7f85cfe  Build Version: 1.6.7995.38578
      For more information, please see http://wiki.ros.org/sw_urdf_exporter -->
-<robot name="gemini_336" xmlns:xacro="http://ros.org/wiki/xacro">
-    <xacro:include filename="gemini_335_336.urdf.xacro"/>
+<robot name="gemini335L" xmlns:xacro="http://ros.org/wiki/xacro">
+    <xacro:include filename="gemini335L_336L.urdf.xacro"/>
     <!-- Define a virtual root link -->
   <link name="base_link"/>
@@ -11,5 +11,5 @@
     <parent link="base_link"/>
     <child link="camera_link"/>
-    <origin xyz="0.01587 0.025 0.0125" rpy="0 0 0"/>
+    <origin xyz="0.011715 0.0475 0.014311" rpy="0 0 0"/>
   </joint>
 </robot>

File: services/robot_container/ros_ws/src/OrbbecSDK_ROS2/orbbec_description/urdf/test_gemini336L.urdf.xacro (robot description, xacro)
@@ -3,6 +3,6 @@
      Commit Version: 1.6.0-4-g7f85cfe  Build Version: 1.6.7995.38578
      For more information, please see http://wiki.ros.org/sw_urdf_exporter -->
-<robot name="gemini_336" xmlns:xacro="http://ros.org/wiki/xacro">
-    <xacro:include filename="gemini_335_336.urdf.xacro"/>
+<robot name="gemini336L" xmlns:xacro="http://ros.org/wiki/xacro">
+    <xacro:include filename="gemini335L_336L.urdf.xacro"/>
     <!-- Define a virtual root link -->
   <link name="base_link"/>
@@ -11,5 +11,5 @@
     <parent link="base_link"/>
     <child link="camera_link"/>
-    <origin xyz="0.01587 0.025 0.0125" rpy="0 0 0"/>
+    <origin xyz="0.011715 0.0475 0.014311" rpy="0 0 0"/>
   </joint>
 </robot>
